Commit message: untermediate commit

File: xv2_description/urdf/xv2_turtle.urdf (robot description, URDF)
Before this commit: robot simple_box, 11 links, 10 joints
Links:
- added link camera_link; collision box size=0.005 0.03 0.03; visual box size=0.005 0.03 0.03
Joints:
- added joint camera_joint: type fixed, parent base_link, child camera_link, origin xyz=1.575 0.4 0.76 rpy=0 -2 0
