Commit message: updated

File: xv2_description/urdf/fake_turtle.urdf (robot description, URDF)
Before this commit: robot simple_box, 18 links, 17 joints
Links:
- link lamp: geometry collision box size=0.05 0.010 0.00001; visual box size=0.0001 0.0001 0.0001
Joints:
- joint light_joint: origin xyz=0.0 0.0 0.0 rpy=0 1.57 0 -> xyz=0.0 0.0 0.0 rpy=1.57 0 0

Commit message: added turtle

File: xv2_description/urdf/fake_turtle.urdf (robot description, URDF)
Before this commit: robot simple_box, 18 links, 17 joints
Links:
- removed link base_link
- removed link camera_link
- removed link fake_turtlebot
- added link box_base_link, mass 1.0; collision box size=0.23 0.23 0.005; visual box size=0.23 0.23 0.005
- added link top_camera_link; collision box size=0.005 0.03 0.03; visual box size=0.005 0.03 0.03
Joints:
- removed joint base_joint
- removed joint camera_joint
- added joint box_base_joint: type fixed, parent base_plate, child box_base_link, origin xyz=0 0 0.01 rpy=0 0 0
- added joint top_camera_joint: type fixed, parent camera_stand, child top_camera_link, origin xyz=0.0 0.0 0.15 rpy=0 0 -2.36
- joint base_standfl_joint: parent fake_turtlebot -> base_link
- joint base_standfr_joint: parent fake_turtlebot -> base_link
- joint base_standrl_joint: parent fake_turtlebot -> base_link
- joint base_standrr_joint: parent fake_turtlebot -> base_link
- joint light_joint: parent camera_link -> top_camera_link
- joint side1_joint: parent base_link -> box_base_link
- joint side2_joint: parent base_link -> box_base_link
- joint side3_joint: parent base_link -> box_base_link
- joint side4_joint: parent base_link -> box_base_link
